File: pcb/rev5/NinoBLE Rev5.kicad_sch (KiCad schematic)
At the start: 14 parts, among them J1 Conn_01x01, J2 Conn_01x01, J3 Conn_01x01, J4 Conn_01x04, J5 TF-01A, J6 Conn_01x01, J7 Conn_01x01, SW1 SW_SPDT, SW2 SW_Push, U1 Pico

Commit message: fixup rev5 pcb files
Parts:
- C1, C2: LCSC Part # (none) -> C28233
- J1, J2, J6, J7: JSCS PN C5157269 -> (none); LCSC Part # (none) -> C5157269
- J4: LSCS PN C5248081 -> (none)
- J5: LCSC Part # (none) -> C91145; LSCS PN C91145 -> (none)
- R1, R2: LCSC Part # (none) -> C17414
- SW1: LCSC Part # (none) -> C221660; LSCS PN C221660 -> (none)
- SW2: LCSC Part # (none) -> C79175; LSCS PN C79175 -> (none)
Changed lines of the file:
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@@
+			)
+		)
+		(property "LCSC Part #" "C28233"
+			(at 30.48 106.68 0)
+			(effects
+				(font
+					(size 1.27 1.27)
+				)
+				(hide yes)
+			)
+		)
+		(property "Part" ""
+			(at 30.48 106.68 0)
+			(effects
+				(font
+					(size 1.27 1.27)
+				)
+				(hide yes)
 			)
 		)
@@
 			)
 		)
-		(property "LSCS PN" "C91145"
+		(property "LCSC Part #" "C91145"
+			(at 76.2 120.65 0)
+			(effects
+				(font
+					(size 1.27 1.27)
+				)
+				(hide yes)
+			)
+		)
+		(property "Part" ""
 			(at 76.2 120.65 0)
 			(effects
@@
 			)
 		)
-		(property "JSCS PN" "C5157269"
-			(at 142.24 24.13 90)
+		(property "LCSC Part #" "C5157269"
+			(at 142.24 24.13 0)
+			(effects
+				(font
+					(size 1.27 1.27)
+				)
+				(hide yes)
+			)
+		)
+		(property "Part" ""
+			(at 142.24 24.13 0)
 			(effects
 				(font
@@
 			)
 		)
-		(property "JSCS PN" "C5157269"
-			(at 144.78 24.13 90)
+		(property "LCSC Part #" "C5157269"
+			(at 144.78 24.13 0)
+			(effects
+				(font
+					(size 1.27 1.27)
+				)
+				(hide yes)
+			)
+		)
+		(property "Part" ""
+			(at 144.78 24.13 0)
 			(effects
 				(font
@@
 			)
 		)
-		(property "LSCS PN" "C79175"
-			(at 179.07 99.06 90)
+		(property "LCSC Part #" "C79175"
+			(at 179.07 99.06 0)
+			(effects
+				(font
+					(size 1.27 1.27)
+				)
+				(hide yes)
+			)
+		)
+		(property "Part" ""
+			(at 179.07 99.06 0)
 			(effects
 				(font
@@
 			)
 		)
-		(property "JSCS PN" "C5157269"
-			(at 147.32 24.13 90)
-			(effects
-				(font
-					(size 1.27 1.27)
-				)
-				(hide yes)
-			)
-		)
 		(property "Field6" ""
 			(at 147.32 24.13 90)
@@
 			)
 		)
+		(property "LCSC Part #" "C5157269"
+			(at 147.32 24.13 0)
+			(effects
+				(font
+					(size 1.27 1.27)
+				)
+				(hide yes)
+			)
+		)
+		(property "Part" ""
+			(at 147.32 24.13 0)
+			(effects
+				(font
+					(size 1.27 1.27)
+				)
+				(hide yes)
+			)
+		)
 		(pin "1"
 		)
@@
 			)
 		)
+		(property "Part" ""
+			(at 127 86.36 0)
+			(effects
+				(font
+					(size 1.27 1.27)
+				)
+				(hide yes)
+			)
+		)
 		(pin "24"
 		)
@@
 			)
 		)
-		(property "LSCS PN" "C221660"
-			(at 167.64 78.74 90)
+		(property "LCSC Part #" "C221660"
+			(at 167.64 78.74 0)
+			(effects
+				(font
+					(size 1.27 1.27)
+				)
+				(hide yes)
+			)
+		)
+		(property "Part" ""
+			(at 167.64 78.74 0)
 			(effects
 				(font
@@
 			)
 		)
+		(property "LCSC Part #" "C28233"
+			(at 41.91 134.62 0)
+			(effects
+				(font
+					(size 1.27 1.27)
+				)
+				(hide yes)
+			)
+		)
+		(property "Part" ""
+			(at 41.91 134.62 0)
+			(effects
+				(font
+					(size 1.27 1.27)
+				)
+				(hide yes)
+			)
+		)
 		(pin "2"
 		)
@@
 			)
 		)
+		(property "LCSC Part #" "C17414"
+			(at 167.64 90.17 0)
+			(effects
+				(font
+					(size 1.27 1.27)
+				)
+				(hide yes)
+			)
+		)
+		(property "Part" ""
+			(at 167.64 90.17 0)
+			(effects
+				(font
+					(size 1.27 1.27)
+				)
+				(hide yes)
+			)
+		)
 		(pin "1"
 		)
@@
 			)
 		)
-		(property "LSCS PN" "C5248081"
+		(property "Part" ""
 			(at 73.66 73.66 0)
 			(effects
@@
 			)
 		)
+		(property "Part" ""
+			(at 87.63 24.13 0)
+			(effects
+				(font
+					(size 1.27 1.27)
+				)
+				(hide yes)
+			)
+		)
 		(pin "1"
 		)
@@
 			)
 		)
+		(property "LCSC Part #" "C17414"
+			(at 41.91 124.46 0)
+			(effects
+				(font
+					(size 1.27 1.27)
+				)
+				(hide yes)
+			)
+		)
+		(property "Part" ""
+			(at 41.91 124.46 0)
+			(effects
+				(font
+					(size 1.27 1.27)
+				)
+				(hide yes)
+			)
+		)
 		(pin "1"
 		)
@@
 			)
 		)
-		(property "JSCS PN" "C5157269"
-			(at 149.86 24.13 90)
-			(effects
-				(font
+		(property "LCSC Part #" "C5157269"
+			(at 149.86 24.13 0)
+			(effects
+				(font
+					(size 1.27 1.27)
+				)
+				(hide yes)
+			)
+		)
+		(property "Part" ""
+			(at 149.86 24.13 0)
+			(effects
+				(font
